File: design/soilsense/soilsense.kicad_sch (KiCad schematic)
At the start: 21 parts, among them Q1 AO3407, Q2 AO3407, U1 TP4056, U2 ESP-01, U3 GXHT30, U4 CapSoilSensor_v1.2, U5 ADS1115IDGS, U6 MCP1700x-330xxTO

Commit message: Finish pcb layout
Parts:
- removed C1: 10uF, symbol Device:C_Polarized
- removed C2: 100nF, Capacitor_THT:C_Radial_D4.0mm_H5.0mm_P1.50mm, symbol Device:C
- removed R5: 4.7K, OptoDevice:R_LDR_5.2x5.2mm_P3.5mm_Horizontal, symbol Device:R
- added C2, C3: 10uF, Capacitor_THT:CP_Radial_D8.0mm_P5.00mm, symbol Device:C_Polarized
- added C4, C5: 100nF, Capacitor_THT:C_Radial_D4.0mm_H5.0mm_P1.50mm, symbol Device:C
- added R1, R8, R9: 100K, Resistor_THT:R_Axial_DIN0207_L6.3mm_D2.5mm_P7.62mm_Horizontal, symbol Device:R
- added R10, R11: 4.7K, Resistor_THT:R_Axial_DIN0207_L6.3mm_D2.5mm_P7.62mm_Horizontal, symbol Device:R
- D1: footprint Diode_THT:D_DO-41_SOD81_P10.16mm_Horizontal -> Diode_THT:D_DO-41_SOD81_P7.62mm_Horizontal
- Q1, Q2: footprint Package_TO_SOT_SMD:SOT-23 -> Connector_PinHeader_2.54mm:PinHeader_1x03_P2.54mm_Vertical
- R2: value 10K -> 100; footprint OptoDevice:R_LDR_5.2x5.2mm_P3.5mm_Horizontal -> Resistor_THT:R_Axial_DIN0207_L6.3mm_D2.5mm_P7.62mm_Horizontal
- R3: value 10K -> 220K; footprint OptoDevice:R_LDR_5.2x5.2mm_P3.5mm_Horizontal -> Resistor_THT:R_Axial_DIN0207_L6.3mm_D2.5mm_P7.62mm_Horizontal
- R4: value 4.7K -> 100K; footprint OptoDevice:R_LDR_5.2x5.2mm_P3.5mm_Horizontal -> Resistor_THT:R_Axial_DIN0207_L6.3mm_D2.5mm_P7.62mm_Horizontal
- R5: renamed from R1; value 10K -> 100K; footprint OptoDevice:R_LDR_5.2x5.2mm_P3.5mm_Horizontal -> Resistor_THT:R_Axial_DIN0207_L6.3mm_D2.5mm_P7.62mm_Horizontal
- R6: value 47K -> 10K; footprint OptoDevice:R_LDR_5.2x5.2mm_P3.5mm_Horizontal -> Resistor_THT:R_Axial_DIN0207_L6.3mm_D2.5mm_P7.62mm_Horizontal
- R7: value 220 -> 10K; footprint OptoDevice:R_LDR_5.2x5.2mm_P3.5mm_Horizontal -> Resistor_THT:R_Axial_DIN0207_L6.3mm_D2.5mm_P7.62mm_Horizontal
- U1: footprint (none) -> symbols:TP4056
- U2: renamed from U4; footprint (none) -> Connector_PinHeader_2.54mm:PinHeader_1x03_P2.54mm_Vertical
- U3: renamed from U5; footprint Package_SO:TSSOP-10_3x3mm_P0.5mm -> Connector_PinHeader_2.54mm:PinHeader_1x10_P2.54mm_Vertical
- U4: renamed from U6; footprint Package_TO_SOT_SMD:SOT-89-3 -> Package_TO_SOT_THT:TO-92
- U5: renamed from U3; footprint Package_DFN_QFN:DFN-6-1EP_2x2mm_P0.5mm_EP0.7x1.6mm -> Connector_PinHeader_2.54mm:PinHeader_1x06_P2.54mm_Vertical
- renumbered C3 to C1, C4 to C6, U2 to U6
Connections:
- net 3.3V: now also C1.2, C6.2, R7.1, U3.1 (VDD), C3.1, C4.1, C5.2, R1.1, R10.1, R11.1; no longer C1.1, C6.1, R2.1, R3.2, U3.8 (VDD)
- net GND: now also C1.1, C6.1, R3.2, R4.1, U3.2 (GND), U3.5 (ADDR), U5.2 (NC), C2.2, C3.2, C4.2, C5.1, R9.2; no longer C1.2, C6.2, U3.1 (ADDR), U3.3 (GND), U5.6 (GND)
- net at U3.9 (AIN2): no longer U5.4 (SDA)
- net 5V: now reaches D1.2 (A), Q1.1 (G), R5.1
- net 5V: now also R8.1
- net at U2.1 (AOUT): now also U3.7 (AIN0); no longer U3.4 (AIN0)
- net at D1.1 (K), Q1.2 (S), U4.2 (VI): now also C2.1
- net at U6.3 (CH_PD): now also R7.2; no longer R2.2
- net at BT1.1 (+), U1.4 (B+): now also R3.1
- net SDA: now reaches U6.4 (GPIO2)
- net SDA: now also U3.4 (SDA), U5.3 (SDA), R10.2; no longer R4.1
- net at U6.5 (RST): now also R6.2; no longer R3.1
- net at U6.1 (UTXD): now also R8.2, R9.1; no longer R7.1
- net SCL: now reaches U6.6 (GPIO0)
- net SCL: now also U3.3 (SCL), U5.4 (SCL), R11.2
- net RX: now reaches U6.8 (URXD)
- net RX: now also R2.1
- new net: Q2.1 (G), R1.2, R2.2
- new net B+: R4.2, U3.8 (AIN1)
- now unconnected: U3.10 (SCL)
- no-connect marks 5 -> 3
Other:
- note added: "ESP8266"
- moved on the sheet: C1, C6, Q2, U2, U3, U4, U5, U6
