File: design/soilsense/soilsense.kicad_sch (KiCad schematic)
At the start: 27 parts, among them Q1 AO3407, Q2 AO3407, U1 TP4056, U2 CapSoilSensor_v1.2, U3 ADS1115IDGS, U4 MCP1700x-330xxTO, U5 GXHT30, U6 ESP-01

Commit message: Add enclosure and refine board layout
Parts:
- C1, C4, C5, C6: footprint Capacitor_THT:C_Radial_D4.0mm_H5.0mm_P1.50mm -> Capacitor_THT:C_Disc_D5.0mm_W2.5mm_P5.00mm
- C2, C3: footprint Capacitor_THT:CP_Radial_D8.0mm_P5.00mm -> Capacitor_THT:CP_Radial_D5.0mm_P2.00mm
- D1: footprint Diode_THT:D_DO-41_SOD81_P7.62mm_Horizontal -> Diode_THT:D_DO-41_SOD81_P10.16mm_Horizontal
- R1, R10, R11, R2, R3, R4, R5, R6, R7, R8, R9: footprint Resistor_THT:R_Axial_DIN0207_L6.3mm_D2.5mm_P7.62mm_Horizontal -> Resistor_THT:R_Axial_DIN0204_L3.6mm_D1.6mm_P5.08mm_Horizontal
- U5: footprint Connector_PinHeader_2.54mm:PinHeader_1x06_P2.54mm_Vertical -> Connector_PinSocket_2.54mm:PinSocket_1x04_P2.54mm_Vertical
Connections:
- net 5V: now also U1.1 (IN+)
